File: Hardware/RS485_Breakout.brd (EAGLE design)
At the start: 22.9 x 27.9 mm, 19 parts, among them U2 RS485SOIC

Commit message: Sch Change
Parts:
- removed JP11: (no value), SparkFun:1X04
- added JP15: STAND-OFF, SparkFun:STAND-OFF
- JP1: value STAND-OFF -> (none); device SparkFun:STAND-OFF -> SparkFun:1X04
- moved JP1 24.7 mm to (7.62, 1.27)
- moved JP10 15.7 mm to (1.27, 21.6)
Connections:
- net 1: now also JP1.4; no longer JP11.4
- net 2: now also JP1.3; no longer JP11.3
- net 3: now also JP1.2; no longer JP11.2
- net 5: now also JP1.1; no longer JP11.1
Changed lines of the file:
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@@
 <layer number="47" name="Measures" color="7" fill="1" visible="no" active="yes"/>
 <layer number="48" name="Document" color="7" fill="1" visible="no" active="yes"/>
-<layer number="49" name="Reference" color="7" fill="1" visible="yes" active="yes"/>
+<layer number="49" name="Reference" color="7" fill="1" visible="no" active="yes"/>
 <layer number="50" name="dxf" color="7" fill="1" visible="no" active="yes"/>
 <layer number="51" name="tDocu" color="6" fill="1" visible="yes" active="yes"/>
@@
 <attribute name="VALUE" value="0.1uF" x="4.953" y="19.431" size="1.778" layer="27" rot="R90" display="off"/>
 </element>
-<element name="JP1" library="SparkFun" package="STAND-OFF" value="STAND-OFF" x="2.54" y="25.4"/>
+<element name="JP15" library="SparkFun" package="STAND-OFF" value="STAND-OFF" x="2.54" y="25.4"/>
 <element name="JP6" library="SparkFun" package="STAND-OFF" value="STAND-OFF" x="2.54" y="2.54"/>
 <element name="JP7" library="SparkFun" package="STAND-OFF" value="STAND-OFF" x="20.32" y="25.4"/>
@@
 <element name="JP9" library="SparkFun" package="1X05" value="" x="2.54" y="19.05" rot="R270"/>
 <element name="JP5" library="SparkFun" package="FIDUCIAL-1X2" value="FIDUCIAL1X2" x="17.78" y="5.08"/>
-<element name="JP10" library="SparkFun" package="FIDUCIAL-1X2" value="FIDUCIAL1X2" x="16.51" y="25.4"/>
-<element name="JP11" library="SparkFun" package="1X04" value="" x="7.62" y="1.27"/>
+<element name="JP10" library="SparkFun" package="FIDUCIAL-1X2" value="FIDUCIAL1X2" x="1.27" y="21.59"/>
+<element name="JP1" library="SparkFun" package="1X04" value="" x="7.62" y="1.27"/>
 <element name="FRAME1" library="SparkFun-Aesthetics" package="CREATIVE_COMMONS" value="FRAME-LETTER" x="-9.379478125" y="-15.24"/>
 <element name="LOGO1" library="SparkFun-Aesthetics" package="OSHW-LOGO-S" value="OSHW-LOGOS" x="8.255" y="25.781"/>
@@
 <signal name="1">
 <contactref element="JP4" pad="1"/>
-<contactref element="JP11" pad="4"/>
+<contactref element="JP1" pad="4"/>
 <wire x1="13.97" y1="2.54" x2="13.97" y2="9.525" width="0.254" layer="1"/>
 <wire x1="15.24" y1="1.27" x2="13.97" y2="2.54" width="0.254" layer="1"/>
@@
 <signal name="2">
 <contactref element="JP4" pad="2"/>
-<contactref element="JP11" pad="3"/>
+<contactref element="JP1" pad="3"/>
 <wire x1="11.43" y1="2.54" x2="11.43" y2="10.795" width="0.254" layer="1"/>
 <wire x1="12.7" y1="1.27" x2="11.43" y2="2.54" width="0.254" layer="1"/>
@@
 <signal name="3">
 <contactref element="JP4" pad="3"/>
-<contactref element="JP11" pad="2"/>
+<contactref element="JP1" pad="2"/>
 <wire x1="14.478" y1="12.065" x2="13.97" y2="12.065" width="0.254" layer="16"/>
 <wire x1="15.875" y1="10.668" x2="14.478" y2="12.065" width="0.254" layer="16"/>
@@
 <signal name="5">
 <contactref element="JP4" pad="6"/>
-<contactref element="JP11" pad="1"/>
+<contactref element="JP1" pad="1"/>
 <wire x1="7.62" y1="12.065" x2="11.43" y2="15.875" width="0.254" layer="16"/>
 <wire x1="7.62" y1="1.27" x2="7.62" y2="12.065" width="0.254" layer="16"/>
